File: SparkFun_Default_KiCad_Setup.kicad_sch (KiCad schematic)
At the start: 18 parts, among them U2 RT9080-3.3

Commit message: Update page settings
Other:
- company: (none) -> SparkFun
Changed lines of the file:
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@@
 	(title_block
 		(title "SparkFun Product (Qwiic)")
-		(date "2024-03-06")
 		(rev "v10")
+		(company "SparkFun")
 		(comment 1 "Designed by: You")
 	)
