File: SparkFun_Default_KiCad_Setup.kicad_sch (KiCad schematic)
At the start: 18 parts, among them U2 RT9080-3.3

Commit message: Update material default to TG135
Parts:
- U2: IMax (none) -> 600mA; VMax 6V -> 5.5V
Changed lines of the file:
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@@
 	(wire
 		(pts
-			(xy 90.17 49.53) (xy 90.17 50.8)
+			(xy 90.17 48.26) (xy 90.17 49.53)
 		)
 		(stroke
@@
 	(wire
 		(pts
-			(xy 77.47 49.53) (xy 77.47 50.8)
+			(xy 77.47 48.26) (xy 77.47 49.53)
 		)
 		(stroke
@@
 	(wire
 		(pts
-			(xy 49.53 40.64) (xy 49.53 41.91)
+			(xy 49.53 40.64) (xy 49.53 43.18)
 		)
 		(stroke
@@
 	(wire
 		(pts
-			(xy 77.47 40.64) (xy 77.47 41.91)
+			(xy 77.47 40.64) (xy 77.47 43.18)
 		)
 		(stroke
@@
 	(wire
 		(pts
-			(xy 90.17 40.64) (xy 90.17 41.91)
+			(xy 90.17 40.64) (xy 90.17 43.18)
 		)
 		(stroke
@@
 	(wire
 		(pts
-			(xy 36.83 49.53) (xy 36.83 50.8)
+			(xy 36.83 48.26) (xy 36.83 49.53)
 		)
 		(stroke
@@
 	(wire
 		(pts
-			(xy 36.83 41.91) (xy 36.83 40.64)
+			(xy 36.83 43.18) (xy 36.83 40.64)
 		)
 		(stroke
@@
 	(wire
 		(pts
-			(xy 49.53 49.53) (xy 49.53 50.8)
+			(xy 49.53 48.26) (xy 49.53 49.53)
 		)
 		(stroke
@@
 			)
 		)
-		(property "Description" ""
+		(property "Description" "Drill holes for mechanically mounting via screws, standoffs, etc."
 			(at 250.19 179.07 0)
 			(effects
@@
 			)
 		)
-		(property "Description" ""
+		(property "Description" "Test Point"
 			(at 27.94 49.53 0)
 			(effects
@@
 	(symbol
 		(lib_id "SparkFun-PowerSymbol:GND")
-		(at 77.47 50.8 0)
+		(at 77.47 49.53 0)
 		(unit 1)
 		(exclude_from_sim no)
@@
 		(fields_autoplaced yes)
 		(property "Reference" "#PWR011"
-			(at 77.47 57.15 0)
+			(at 77.47 55.88 0)
 			(effects
 				(font
@@
 		)
 		(property "Value" "GND"
-			(at 77.47 54.61 0)
+			(at 77.47 53.34 0)
 			(do_not_autoplace yes)
 			(effects
@@
 		)
 		(property "Footprint" ""
-			(at 77.47 50.8 0)
+			(at 77.47 49.53 0)
 			(effects
 				(font
@@
 		)
 		(property "Datasheet" ""
-			(at 77.47 50.8 0)
-			(effects
-				(font
-					(size 1.27 1.27)
-				)
-				(hide yes)
-			)
-		)
-		(property "Description" ""
-			(at 77.47 50.8 0)
+			(at 77.47 49.53 0)
+			(effects
+				(font
+					(size 1.27 1.27)
+				)
+				(hide yes)
+			)
+		)
+		(property "Description" "Power symbol creates a global label with name \"GND\" , ground"
+			(at 77.47 49.53 0)
 			(effects
 				(font
@@
 			)
 		)
-		(property "Description" ""
+		(property "Description" "Unpolarized capacitor"
 			(at 77.47 45.72 0)
 			(effects
@@
 			)
 		)
-		(property "Description" ""
+		(property "Description" "Unpolarized capacitor"
 			(at 90.17 45.72 0)
 			(effects
@@
 			)
 		)
-		(property "Description" ""
+		(property "Description" "Drill holes for mechanically mounting via screws, standoffs, etc."
 			(at 254 179.07 0)
 			(effects
@@
 			)
 		)
-		(property "Description" ""
+		(property "Description" "Drill holes for mechanically mounting via screws, standoffs, etc."
 			(at 250.19 175.26 0)
 			(effects
@@
 			)
 		)
-		(property "Description" ""
+		(property "Description" "Power symbol creates a global label with name \"GND\" , ground"
 			(at 27.94 50.8 0)
 			(effects
@@
 			)
 		)
-		(property "Description" ""
+		(property "Description" "Power symbol creates a global label with name \"GND\" , ground"
 			(at 68.58 52.07 0)
 			(effects
@@
 	(symbol
 		(lib_id "SparkFun-PowerSymbol:GND")
-		(at 49.53 50.8 0)
+		(at 49.53 49.53 0)
 		(unit 1)
 		(exclude_from_sim no)
@@
 		(fields_autoplaced yes)
 		(property "Reference" "#PWR06"
-			(at 49.53 57.15 0)
+			(at 49.53 55.88 0)
 			(effects
 				(font
@@
 		)
 		(property "Value" "GND"
-			(at 49.53 54.61 0)
+			(at 49.53 53.34 0)
 			(do_not_autoplace yes)
 			(effects
@@
 		)
 		(property "Footprint" ""
-			(at 49.53 50.8 0)
+			(at 49.53 49.53 0)
 			(effects
 				(font
@@
 		)
 		(property "Datasheet" ""
-			(at 49.53 50.8 0)
-			(effects
-				(font
-					(size 1.27 1.27)
-				)
-				(hide yes)
-			)
-		)
-		(property "Description" ""
-			(at 49.53 50.8 0)
+			(at 49.53 49.53 0)
+			(effects
+				(font
+					(size 1.27 1.27)
+				)
+				(hide yes)
+			)
+		)
+		(property "Description" "Power symbol creates a global label with name \"GND\" , ground"
+			(at 49.53 49.53 0)
 			(effects
 				(font
@@
 			)
 		)
-		(property "Description" ""
+		(property "Description" "Fiducial Marker"
 			(at 262.89 179.07 0)
 			(effects
@@
 			)
 		)
-		(property "Description" ""
+		(property "Description" "Drill holes for mechanically mounting via screws, standoffs, etc."
 			(at 254 175.26 0)
 			(effects
@@
 			)
 		)
-		(property "Description" ""
+		(property "Description" "Fiducial Marker"
 			(at 259.08 179.07 0)
 			(effects
@@
 	(symbol
 		(lib_id "SparkFun-PowerSymbol:GND")
-		(at 90.17 50.8 0)
+		(at 90.17 49.53 0)
 		(unit 1)
 		(exclude_from_sim no)
@@
 		(fields_autoplaced yes)
 		(property "Reference" "#PWR012"
-			(at 90.17 57.15 0)
+			(at 90.17 55.88 0)
 			(effects
 				(font
@@
 		)
 		(property "Value" "GND"
-			(at 90.17 54.61 0)
+			(at 90.17 53.34 0)
 			(do_not_autoplace yes)
 			(effects
@@
 		)
 		(property "Footprint" ""
-			(at 90.17 50.8 0)
+			(at 90.17 49.53 0)
 			(effects
 				(font
@@
 		)
 		(property "Datasheet" ""
-			(at 90.17 50.8 0)
-			(effects
-				(font
-					(size 1.27 1.27)
-				)
-				(hide yes)
-			)
-		)
-		(property "Description" ""
-			(at 90.17 50.8 0)
+			(at 90.17 49.53 0)
+			(effects
+				(font
+					(size 1.27 1.27)
+				)
+				(hide yes)
+			)
+		)
+		(property "Description" "Power symbol creates a global label with name \"GND\" , ground"
+			(at 90.17 49.53 0)
 			(effects
 				(font
@@
 			)
 		)
-		(property "Description" ""
+		(property "Description" "Power symbol creates a global label with name \"3.3V\""
 			(at 77.47 39.37 0)
 			(effects
@@
 			)
 		)
-		(property "Description" ""
+		(property "Description" "Fiducial Marker"
 			(at 259.08 175.26 0)
 			(effects
@@
 			)
 		)
-		(property "Description" ""
+		(property "Description" "Unpolarized capacitor"
 			(at 49.53 45.72 0)
 			(effects
@@
 			)
 		)
-		(property "Description" ""
+		(property "Description" "Power symbol creates a global label with name \"VCC\""
 			(at 49.53 39.37 0)
 			(effects
@@
 	(symbol
 		(lib_id "SparkFun-PowerSymbol:GND")
-		(at 36.83 50.8 0)
+		(at 36.83 49.53 0)
 		(unit 1)
 		(exclude_from_sim no)
@@
 		(fields_autoplaced yes)
 		(property "Reference" "#PWR05"
-			(at 36.83 57.15 0)
+			(at 36.83 55.88 0)
 			(effects
 				(font
@@
 		)
 		(property "Value" "GND"
-			(at 36.83 54.61 0)
+			(at 36.83 53.34 0)
 			(do_not_autoplace yes)
 			(effects
@@
 		)
 		(property "Footprint" ""
-			(at 36.83 50.8 0)
+			(at 36.83 49.53 0)
 			(effects
 				(font
@@
 		)
 		(property "Datasheet" ""
-			(at 36.83 50.8 0)
-			(effects
-				(font
-					(size 1.27 1.27)
-				)
-				(hide yes)
-			)
-		)
-		(property "Description" ""
-			(at 36.83 50.8 0)
+			(at 36.83 49.53 0)
+			(effects
+				(font
+					(size 1.27 1.27)
+				)
+				(hide yes)
+			)
+		)
+		(property "Description" "Power symbol creates a global label with name \"GND\" , ground"
+			(at 36.83 49.53 0)
 			(effects
 				(font
@@
 			)
 		)
-		(property "Description" ""
+		(property "Description" "Test Point"
 			(at 36.83 39.37 0)
 			(effects
@@
 		(fields_autoplaced yes)
 		(property "Reference" "U2"
+			(at 68.58 31.75 0)
+			(effects
+				(font
+					(size 1.27 1.27)
+				)
+			)
+		)
+		(property "Value" "RT9080-3.3"
 			(at 68.58 34.29 0)
-			(effects
-				(font
-					(size 1.27 1.27)
-				)
-			)
-		)
-		(property "Value" "RT9080-3.3"
-			(at 68.58 36.83 0)
 			(effects
 				(font
@@
 			)
 		)
-		(property "Description" ""
+		(property "Description" "600mA low dropout linear regulator, with enable pin, 3.8V-6V input voltage range, 3.3V fixed positive output, SOT-23-5"
 			(at 68.58 43.18 0)
 			(effects
@@
 			)
 		)
-		(property "VMax" "6V"
+		(property "VMax" "5.5V"
 			(at 68.58 62.23 0)
 			(effects
@@
 			)
 		)
+		(property "IMax" "600mA"
+			(at 68.58 36.83 0)
+			(effects
+				(font
+					(size 1.27 1.27)
+				)
+			)
+		)
 		(pin "1"
 		)
@@
 			)
 		)
-		(property "Description" ""
+		(property "Description" "Unpolarized capacitor"
 			(at 36.83 45.72 0)
 			(effects
@@
 			)
 		)
-		(property "Description" ""
+		(property "Description" "Fiducial Marker"
 			(at 262.89 175.26 0)
 			(effects
