File: SparkFun_Default_KiCad_Setup.kicad_pcb (KiCad board)
At the start: 4 copper layers, 50.8 x 50.8 mm, 18 parts, among them U2 RT9080-3.3

Commit message: Set pad_to_mask_clearance to 0.05mm
Other:
- rule pad_to_mask_clearance: 0 -> 0.05
Changed lines of the file:
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@@
 			(dielectric_constraints no)
 		)
-		(pad_to_mask_clearance 0)
+		(pad_to_mask_clearance 0.05)
 		(allow_soldermask_bridges_in_footprints no)
 		(aux_axis_origin 115.57 124.46)
@@
 		(layer "F.Cu")
 		(at 215.265 168.91)
-		(tags "Creative Commons License")
+		(tags "SparkFun Creative Commons License")
 		(property "Reference" "G3"
 			(at 0 -5.08 0)
@@
 			)
 		)
-		(sheetname "Root")
-		(sheetfile "SparkFun_Default_KiCad_Setup.kicad_sch")
 		(attr exclude_from_bom)
-		(fp_text user "Released under the Creative Commons Attribution Share-Alike 4.0 License"
-			(at 0 -1.27 0)
+		(fp_text user " https://creativecommons.org/licenses/by-sa/4.0/"
+			(at 0 1.27 0)
 			(layer "User.1")
 			(effects
@@
 			)
 		)
-		(fp_text user " https://creativecommons.org/licenses/by-sa/4.0/"
-			(at 0 1.27 0)
+		(fp_text user "Released under the Creative Commons Attribution Share-Alike 4.0 License"
+			(at 0 -1.27 0)
 			(layer "User.1")
 			(effects
@@
 		(layer "F.Cu")
 		(at 141.605 106.68)
+		(tags "SparkFun")
 		(property "Reference" "U2"
 			(at 0 -2 0)
@@
 			)
 		)
-		(property ki_fp_filters "SOT?23?5*")
-		(sheetname "Root")
-		(sheetfile "SparkFun_Default_KiCad_Setup.kicad_sch")
 		(fp_line
 			(start -0.4294 -1.27)
@@
 			(thermal_bridge_angle 0)
 		)
+		(model "${SPARKFUN_KICAD_LIBRARY}/Footprints/SparkFun-3D-models/Semiconductor-Standard/SOT-23-5.step"
+			(offset
+				(xyz 0 0 0)
+			)
+			(scale
+				(xyz 1 1 1)
+			)
+			(rotate
+				(xyz 0 0 0)
+			)
+		)
 	)
 	(footprint "SparkFun-Connector:TestPoint-0.75mm"
 		(layer "F.Cu")
 		(at 138.43 103.505)
+		(tags "SparkFun")
 		(property "Reference" "TP2"
 			(at 0 -1.016 0)
@@
 			)
 		)
-		(property ki_fp_filters "Pin* Test*")
-		(sheetname "Root")
-		(sheetfile "SparkFun_Default_KiCad_Setup.kicad_sch")
 		(fp_circle
 			(center 0 0)
@@
 		(layer "F.Cu")
 		(at 163.83 121.92)
+		(tags "SparkFun")
 		(property "Reference" "ST4"
 			(at 0 -2.032 0)
@@
 			)
 		)
-		(property ki_fp_filters "Fiducial*")
-		(sheetname "Root")
-		(sheetfile "SparkFun_Default_KiCad_Setup.kicad_sch")
 		(fp_circle
 			(center 0 0)
@@
 		(at 165.1 118.11)
 		(descr "Circular Fiducial, 0.5mm bare copper, 1mm soldermask opening (Level C)")
-		(tags "fiducial")
+		(tags "SparkFun fiducial")
 		(property "Reference" "FID4"
 			(at 0 -1.5 0)
@@
 			)
 		)
-		(property ki_fp_filters "Fiducial*")
-		(sheetname "Root")
-		(sheetfile "SparkFun_Default_KiCad_Setup.kicad_sch")
 		(attr smd)
 		(fp_circle
@@
 		(at 121.92 74.93)
 		(descr "Circular Fiducial, 0.5mm bare copper, 1mm soldermask opening (Level C)")
-		(tags "fiducial")
+		(tags "SparkFun fiducial")
 		(property "Reference" "FID1"
 			(at 0 -1.5 0)
@@
 			)
 		)
-		(property ki_fp_filters "Fiducial*")
-		(sheetname "Root")
-		(sheetfile "SparkFun_Default_KiCad_Setup.kicad_sch")
 		(attr smd)
 		(fp_circle
@@
 		(layer "F.Cu")
 		(at 138.43 106.68 -90)
-		(tags "capacitor")
+		(tags "SparkFun capacitor")
 		(property "Reference" "C3"
 			(at 0 -1.43 90)
@@
 			)
 		)
-		(property ki_fp_filters "C_*")
-		(sheetname "Root")
-		(sheetfile "SparkFun_Default_KiCad_Setup.kicad_sch")
 		(attr smd)
 		(fp_line
@@
 			(pintype "passive")
 		)
-		(model "${KICAD6_3DMODEL_DIR}/Capacitor_SMD.3dshapes/C_0603_1608Metric.wrl"
+		(model "${SPARKFUN_KICAD_LIBRARY}/Footprints/SparkFun-3D-models/Capacitor/C_0603_1608Metric.step"
 			(offset
 				(xyz 0 0 0)
@@
 		(layer "F.Cu")
 		(at 163.83 76.2)
+		(tags "SparkFun")
 		(property "Reference" "ST3"
 			(at 0 -2.032 0)
@@
 			)
 		)
-		(property ki_fp_filters "Fiducial*")
-		(sheetname "Root")
-		(sheetfile "SparkFun_Default_KiCad_Setup.kicad_sch")
 		(fp_circle
 			(center 0 0)
@@
 		(layer "F.Cu")
 		(at 141.605 80.01)
+		(tags "SparkFun")
 		(property "Reference" "G***"
 			(at 0 -3.8 0)
@@
 		)
 		(group ""
-			(members "1290c26e-57ae-4191-a591-3894405e5662" "22b51b58-d84d-4529-9b44-37ff6d530403"
-				"62bd23c4-a50a-4fac-9d1e-242acbe10b58" "631636e7-b788-404d-88ee-5fa0035e2be3"
-				"743e17b5-8780-47e7-9122-03920230874b" "81fc986d-0167-4f8d-8dee-f7dca86a600f"
-				"8a355bca-cd48-4181-a33d-4d5d54be9967" "d591b2a8-ec86-4c61-b835-ad54105cd10d"
-				"dd31932a-8370-44de-9894-aa622000e827"
+			(members "14362964-c3b7-4895-9424-a66e9f5fe93e" "3ad70b15-59d9-4f65-b0a2-73efb54734e3"
+				"3b7dd05a-f9ac-45ae-811c-da3f1f158997" "6ab5057b-e6c1-4a56-bac3-c844af29af9d"
+				"a26fabc5-2cdf-4e89-8180-9b5f547cba7d" "c8d1802f-9481-426f-98db-23b98f4dd98a"
+				"d0cf64a4-81eb-4a66-9896-ad7d5687dc52" "e1c77c63-1fac-4865-92eb-27c174408ec0"
+				"f4b3ceab-359e-4a15-81ba-a11fc8ca4b5a"
 			)
 		)
@@
 		(layer "F.Cu")
 		(at 146.685 106.68 -90)
-		(tags "capacitor")
+		(tags "SparkFun capacitor")
 		(property "Reference" "C5"
 			(at 0 -1.43 90)
@@
 			)
 		)
-		(property ki_fp_filters "C_*")
-		(sheetname "Root")
-		(sheetfile "SparkFun_Default_KiCad_Setup.kicad_sch")
 		(attr smd)
 		(fp_line
@@
 			(pintype "passive")
 		)
-		(model "${KICAD6_3DMODEL_DIR}/Capacitor_SMD.3dshapes/C_0603_1608Metric.wrl"
+		(model "${SPARKFUN_KICAD_LIBRARY}/Footprints/SparkFun-3D-models/Capacitor/C_0603_1608Metric.step"
 			(offset
 				(xyz 0 0 0)
@@
 		(layer "F.Cu")
 		(at 138.43 109.22)
+		(tags "SparkFun")
 		(property "Reference" "TP1"
 			(at 0 -1.016 0)
@@
 			)
 		)
-		(property ki_fp_filters "Pin* Test*")
-		(sheetname "Root")
-		(sheetfile "SparkFun_Default_KiCad_Setup.kicad_sch")
 		(fp_circle
 			(center 0 0)
@@
 		(layer "F.Cu")
 		(at 136.525 106.68 -90)
-		(tags "capacitor")
+		(tags "SparkFun capacitor")
 		(property "Reference" "C2"
 			(at 0 -1.43 90)
@@
 			)
 		)
-		(property ki_fp_filters "C_*")
-		(sheetname "Root")
-		(sheetfile "SparkFun_Default_KiCad_Setup.kicad_sch")
 		(attr smd)
 		(fp_line
@@
 			(pintype "passive")
 		)
-		(model "${KICAD6_3DMODEL_DIR}/Capacitor_SMD.3dshapes/C_0603_1608Metric.wrl"
+		(model "${SPARKFUN_KICAD_LIBRARY}/Footprints/SparkFun-3D-models/Capacitor/C_0603_1608Metric.step"
 			(offset
 				(xyz 0 0 0)
@@
 		(layer "F.Cu")
 		(at 118.11 76.2)
+		(tags "SparkFun")
 		(property "Reference" "ST1"
 			(at 0 -2.032 0)
@@
 			)
 		)
-		(property ki_fp_filters "Fiducial*")
-		(sheetname "Root")
-		(sheetfile "SparkFun_Default_KiCad_Setup.kicad_sch")
 		(fp_circle
 			(center 0 0)
@@
 		(at 144.78 106.68 -90)
 		(descr "Capacitor SMD 0402 (1005 Metric), square (rectangular) end terminal, IPC_7351 nominal, (Body size source: IPC-SM-782 page 76, https://www.pcb-3d.com/wordpress/wp-content/uploads/ipc-sm-782a_amendment_1_and_2.pdf), generated with kicad-footprint-generator")
-		(tags "capacitor")
+		(tags "SparkFun capacitor")
 		(property "Reference" "C4"
 			(at 0 -1.16 90)
@@
 			)
 		)
-		(property ki_fp_filters "C_*")
-		(sheetname "Root")
-		(sheetfile "SparkFun_Default_KiCad_Setup.kicad_sch")
 		(attr smd)
 		(fp_line
@@
 			(pintype "passive")
 		)
-		(model "${KICAD6_3DMODEL_DIR}/Capacitor_SMD.3dshapes/C_0402_1005Metric.wrl"
+		(model "${SPARKFUN_KICAD_LIBRARY}/Footprints/SparkFun-3D-models/Capacitor/C_0402_1005Metric.step"
 			(offset
 				(xyz 0 0 0)
@@
 		(layer "F.Cu")
 		(at 118.11 121.92)
+		(tags "SparkFun")
 		(property "Reference" "ST2"
 			(at 0 -2.032 0)
@@
 			)
 		)
-		(property ki_fp_filters "Fiducial*")
-		(sheetname "Root")
-		(sheetfile "SparkFun_Default_KiCad_Setup.kicad_sch")
 		(fp_circle
 			(center 0 0)
@@
 		(at 121.92 74.93 180)
 		(descr "Circular Fiducial, 0.5mm bare copper, 1mm soldermask opening (Level C)")
-		(tags "fiducial")
+		(tags "SparkFun fiducial")
 		(property "Reference" "FID3"
 			(at 0 1.5 0)
@@
 			)
 		)
-		(property ki_fp_filters "Fiducial*")
-		(sheetname "Root")
-		(sheetfile "SparkFun_Default_KiCad_Setup.kicad_sch")
 		(attr smd)
 		(fp_circle
@@
 		(at 165.1 118.11 180)
 		(descr "Circular Fiducial, 0.5mm bare copper, 1mm soldermask opening (Level C)")
-		(tags "fiducial")
+		(tags "SparkFun fiducial")
 		(property "Reference" "FID2"
 			(at 0 1.5 0)
@@
 			)
 		)
-		(property ki_fp_filters "Fiducial*")
-		(sheetname "Root")
-		(sheetfile "SparkFun_Default_KiCad_Setup.kicad_sch")
 		(attr smd)
 		(fp_circle
@@
 		(layer "B.Cu")
 		(at 128.27 107.95 180)
+		(tags "SparkFun")
 		(property "Reference" "G***"
 			(at 0 3.8 0)
@@
 		)
 		(group ""
-			(members "0b546f01-1637-4bc7-bfd2-04961f04b3cf" "10a8437a-4088-40f6-b702-98e4dd5e2a21"
-				"120a4d1e-b3cd-44cd-a996-1162bf6f05c6" "51c847fb-c48d-409a-baea-1f1542a0a4e2"
-				"65503c14-84a6-4c56-a457-99940475921a" "6eb1913b-bcea-46f7-b9ba-4c01bad7a9a5"
-				"94ba66bb-7cfc-423d-92c2-91ab8064b60e" "96ab9529-5772-4ad1-a9ad-e83f573706e4"
-				"fed07d67-42e6-4142-b92b-05c71ba79ccc"
+			(members "2f1b36f7-2356-4ac1-8e64-2e6bf1c8339c" "39b472e4-6125-437a-ab02-b49d6b173870"
+				"84a940c5-076f-4d5d-9688-5feaa38c246d" "84fd0a9c-fdf9-464f-b14d-0f6baa0e7759"
+				"88182172-5da0-4276-a981-d0d85582db47" "8a6477b6-998a-40c2-a5ea-7eb609062c5a"
+				"b8cf335b-fe64-42d3-a51a-4311cdc2c858" "bd31b5d9-97ec-436b-a50d-6bd2a13263c8"
+				"fb5ebd34-0095-4425-aa4f-a0462d998cf6"
 			)
 		)
@@
 		)
 		(height -3.81)
-		(gr_text "2000 mils"
+		(gr_text "50.8 mm"
 			(at 140.97 68.7 0)
 			(layer "Dwgs.User")
@@
 		)
 		(height 2.54)
-		(gr_text "100 mils"
+		(gr_text "2.5 mm"
 			(at 167.76 123.19 90)
 			(layer "Dwgs.User")
@@
 		)
 		(height 2.54)
-		(gr_text "100 mils"
+		(gr_text "2.5 mm"
 			(at 116.84 125.85 0)
 			(layer "Dwgs.User")
@@
 		)
 		(height -3.81)
-		(gr_text "2000 mils"
+		(gr_text "50.8 mm"
 			(at 110.61 99.06 90)
 			(layer "Dwgs.User")

Commit message: Layer rename
Other:
- board text added: "Controlled Impedance: JLC04161H-7628"
- board text removed: "Controlled Impedance: JLC7628"
Changed lines of the file:
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@@
 	(layers
 		(0 "F.Cu" signal)
-		(1 "In1.Cu" signal)
-		(2 "In2.Cu" signal)
-		(31 "B.Cu" signal)
+		(1 "In1.Cu" signal "L2.Cu")
+		(2 "In2.Cu" signal "L3.Cu")
+		(31 "B.Cu" jumper)
 		(34 "B.Paste" user)
 		(35 "F.Paste" user)
@@
 		(38 "B.Mask" user)
 		(39 "F.Mask" user)
-		(40 "Dwgs.User" user "User.Drawings")
-		(41 "Cmts.User" user "User.Comments")
-		(42 "Eco1.User" user "User.Eco1")
-		(43 "Eco2.User" user "User.Eco2")
+		(40 "Dwgs.User" user "Measures")
+		(41 "Cmts.User" user "V-score")
+		(42 "Eco1.User" user "Fab.Info")
+		(43 "Eco2.User" user "License.Info")
 		(44 "Edge.Cuts" user)
 		(45 "Margin" user)
 		(46 "B.CrtYd" user "B.Courtyard")
 		(47 "F.CrtYd" user "F.Courtyard")
-		(48 "B.Fab" user)
-		(49 "F.Fab" user)
-		(50 "User.1" user)
+		(48 "B.Fab" user "B.Outlines")
+		(49 "F.Fab" user "F.Outlines")
+		(50 "User.1" user "Milling")
+		(51 "User.2" user "Design.Info")
+		(52 "User.3" user "Board.Properties")
+		(53 "User.4" user "Selective.Solder")
+		(54 "User.5" user "Enclsoure.Info")
 	)
 	(setup
@@
 		(fp_text user " https://creativecommons.org/licenses/by-sa/4.0/"
 			(at 0 1.27 0)
-			(layer "User.1")
+			(layer "Eco2.User")
 			(effects
 				(font
@@
 		(fp_text user "Released under the Creative Commons Attribution Share-Alike 4.0 License"
 			(at 0 -1.27 0)
-			(layer "User.1")
+			(layer "Eco2.User")
 			(effects
 				(font
@@
 	(gr_text "No Clean Process"
 		(at 226.06 182.88 0)
-		(layer "F.Fab")
+		(layer "Eco1.User")
 		(effects
 			(font
@@
 	(gr_text "Inner Copper Weight: 0.5oz"
 		(at 226.06 186.69 0)
-		(layer "F.Fab")
+		(layer "Eco1.User")
 		(effects
 			(font
@@
 	(gr_text "Layers: 4"
 		(at 195.530892 182.88 0)
-		(layer "F.Fab")
+		(layer "Eco1.User")
 		(effects
 			(font
@@
 	(gr_text "Silkscreen Color: White"
 		(at 195.58 180.975 0)
-		(layer "F.Fab")
+		(layer "Eco1.User")
 		(effects
 			(font
@@
 	(gr_text "Solder Mask: Red"
 		(at 195.58 179.07 0)
-		(layer "F.Fab")
+		(layer "Eco1.User")
 		(effects
 			(font
@@
 	(gr_text "Material: TG155"
 		(at 226.06 180.975 0)
-		(layer "F.Fab")
+		(layer "Eco1.User")
 		(effects
 			(font
@@
 		)
 	)
-	(gr_text "Controlled Impedance: JLC7628"
+	(gr_text "Controlled Impedance: JLC04161H-7628"
 		(at 226.06 179.07 0)
-		(layer "F.Fab")
+		(layer "Eco1.User")
 		(effects
 			(font
@@
 	(gr_text "Outer Copper Weight: 1oz"
 		(at 226.06 184.785 0)
-		(layer "F.Fab")
+		(layer "Eco1.User")
 		(effects
 			(font
@@
 	(gr_text "Thickness: 1.6mm"
 		(at 195.58 184.785 0)
-		(layer "F.Fab")
+		(layer "Eco1.User")
 		(effects
 			(font
@@
 	(gr_text "Finish: ENIG"
 		(at 195.58 186.69 0)
-		(layer "F.Fab")
+		(layer "Eco1.User")
 		(effects
 			(font
@@
 	(gr_text "Ordering Notes"
 		(at 189.23 175.895 0)
-		(layer "F.Fab")
+		(layer "Eco1.User")
 		(effects
 			(font
@@
 		)
 		(height -3.81)
-		(gr_text "50.8 mm"
+		(gr_text "2000 mils"
 			(at 140.97 68.7 0)
 			(layer "Dwgs.User")
@@
 		)
 		(height 2.54)
-		(gr_text "2.5 mm"
+		(gr_text "100 mils"
 			(at 167.76 123.19 90)
 			(layer "Dwgs.User")
@@
 		)
 		(height 2.54)
-		(gr_text "2.5 mm"
+		(gr_text "100 mils"
 			(at 116.84 125.85 0)
 			(layer "Dwgs.User")
@@
 		)
 		(height -3.81)
-		(gr_text "50.8 mm"
+		(gr_text "2000 mils"
 			(at 110.61 99.06 90)
 			(layer "Dwgs.User")
