File: Example-Basic Board/SparkFun_Basic_Board_Example.kicad_sch (KiCad schematic)
At the start: 20 parts, among them J1 Qwiic_RA, U2 RT9080-3.3

Commit message: Update examples with latest parts
Parts:
- C5: PROD_ID CAP-11015 -> CAP-25001
- J1: footprint SparkFun-Connector:JST_SMD_1.0mm-4_Black -> SparkFun-Connector:JST_1x04_P1.0mm_Horizontal_SMD; symbol SparkFun-Connector:Qwiic_Right_Angle -> SparkFun-Connector:Qwiic_Horizontal
Other:
- moved on the sheet: C2, C3, C5, J1, TP1, TP2
