File: Example-Qwiic Micro Breakout/SparkFun_Example_Micro.kicad_pcb (KiCad board)
At the start: 2 copper layers, 19 x 7.6 mm, 27 parts, among them J1 PTH_1x1mm, J2 Qwiic_RA, J5 PTH_1x1mm

Commit message: Remove duplicate files
Parts:
- removed kibuzzard-6841DB2D: G***, kibuzzard-6841DB2D
- removed kibuzzard-6846F956: G***, kibuzzard-6846F956
- removed kibuzzard-6846F976: G***, kibuzzard-6846F976
- added C4: 10uF, SparkFun-Capacitor:C_0402_1005Metric, F.Cu at (134.4, 109.5)
- added JP3: ADDR, SparkFun-Jumper:Jumper_2_NO, B.Cu at (130.9, 109.5)
- added R2: 10k, SparkFun-Resistor:R_0402_1005Metric, F.Cu at (130.6, 109.5)
- added U1: LIS3DH, SparkFun-Sensor:ST_LGA-16_3x3mm_P0.5mm_5x3, F.Cu at (132.2, 107.0)
- added kibuzzard-6841DC10: G***, kibuzzard-6841DC10, F.Cu at (128.3, 107.0)
- added kibuzzard-6841DC10: G***, kibuzzard-6841DC10, B.Cu at (128.3, 107.0)
- added kibuzzard-6841DC42: G***, kibuzzard-6841DC42, B.Cu at (130.9, 106.6)
- added kibuzzard-6841DC70: G***, kibuzzard-6841DC70, B.Cu at (132.9, 104.5)
- added kibuzzard-68489829: G***, kibuzzard-68489829, F.Cu at (126.1, 109.5)
- added kibuzzard-68489831: G***, kibuzzard-68489831, F.Cu at (126.2, 104.6)
- D1: footprint SparkFun-LED:LED_0402_1005Metric -> SparkFun-LED:LED_0402_1005Metric_Red
- J1, J5: footprint SparkFun-Connector:1x01_PTH_1x1mm -> SparkFun-Connector:1x01_1x1mm
- moved JP1 3.40 mm to (135.4, 104.4)
Connections:
- J1 pad 1: INT -> INT1
Routing:
- net 3.3V: track 0.00 -> 26.6 mm, vias 0 -> 2
- net SDA: track 0.06 -> 14.4 mm, vias 0 -> 1
- net SCL: track 0.00 -> 11.3 mm, vias 0 -> 1
- net ADDR/SDO: track 0.00 -> 9.43 mm, vias 0 -> 2
- net Net-(JP2-C): track 0.00 -> 4.61 mm, vias 0 -> 1
- net Net-(JP2-A): track 0.00 -> 4.43 mm, vias 0 -> 1
- net INT1: track 0.00 -> 4.39 mm
- net Net-(JP1-A): track 0.00 -> 1.41 mm, vias 0 -> 1
- net GND: vias 0 -> 6

Commit message: Add axis labels
Parts:
- removed FID1, FID2: Fiducial_0.5mm, SparkFun-Aesthetic:Fiducial_0.5mm_Mask1mm
- removed kibuzzard-6841DC42: G***, kibuzzard-6841DC42
- removed kibuzzard-6841DC70: G***, kibuzzard-6841DC70
- removed kibuzzard-68489829: G***, kibuzzard-68489829
- removed kibuzzard-68489831: G***, kibuzzard-68489831
- added kibuzzard-685702DA: G***, kibuzzard-685702DA, B.Cu at (132.8, 104.5)
- added kibuzzard-6857032D: G***, kibuzzard-6857032D, B.Cu at (134.1, 109.5)
- added kibuzzard-685705B3: G***, kibuzzard-685705B3, F.Cu at (135.3, 104.1)
- added kibuzzard-685705E6: G***, kibuzzard-685705E6, F.Cu at (129.3, 107.6)
- added kibuzzard-685705E9: G***, kibuzzard-685705E9, F.Cu at (136.0, 109.9)
- added kibuzzard-68570718: G***, kibuzzard-68570718, F.Cu at (126.1, 109.5)
- added kibuzzard-68570728: G***, kibuzzard-68570728, F.Cu at (126.4, 104.5)
- JP1: value LED -> ~
- JP2: value I2C -> ~
- JP3: value ADDR -> ~
- moved G*** 5.91 mm to (138.5, 109.9)
- moved Ref** 5.48 mm to (125.8, 104.5)
- moved FID3 2.55 mm to (123.9, 103.8)
- moved R6 2.25 mm to (135.3, 105.7), turned to 90 degrees
- moved R1 1.81 mm to (135.3, 107.8)
- moved FID4 1.08 mm to (140.1, 108.6)
- moved C3 0.32 mm to (132.5, 109.9)
- moved C4 0.32 mm to (134.4, 109.9)
- moved R2 0.32 mm to (130.6, 109.9)
- moved TP5 0.25 mm to (141.0, 104.1)
- moved TP6 0.25 mm to (141.0, 106.0)
- moved TP7 0.25 mm to (141.0, 107.9)
- moved TP8 0.25 mm to (141.0, 109.9)
- moved J2 0.15 mm to (137.2, 107.0)
- moved G*** 0.13 mm to (133.4, 107.0)
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Connections:
- net ADDR/SDO renamed ADR/SDO
Routing:
- net GND: track 0.00 -> 6.28 mm, vias 6 -> 4
- net SDA: track 14.4 -> 11.6 mm, vias 1 -> 3
- net SCL: track 11.3 -> 8.73 mm
- net 3.3V: track 26.6 -> 24.7 mm, vias 2 -> 1
- net ADR/SDO: track 9.43 -> 10.5 mm, vias 2 -> 1
- net INT1: track 4.39 -> 4.61 mm, vias 0 -> 1
Other:
- board text added: "v10"

Commit message: Make labels and text follow standard
Parts:
- removed kibuzzard-6841DC10 (x2): G***, kibuzzard-6841DC10
- removed kibuzzard-6841DC9E: G***, kibuzzard-6841DC9E
- removed kibuzzard-685702DA: G***, kibuzzard-685702DA
- removed kibuzzard-6857032D: G***, kibuzzard-6857032D
- removed kibuzzard-685705B3: G***, kibuzzard-685705B3
- removed kibuzzard-685705E6: G***, kibuzzard-685705E6
- removed kibuzzard-685705E9: G***, kibuzzard-685705E9
- removed kibuzzard-68570718: G***, kibuzzard-68570718
- removed kibuzzard-68570728: G***, kibuzzard-68570728
- added kibuzzard-689A65D0: G***, kibuzzard-689A65D0, F.Cu at (126.3, 109.5)
- added kibuzzard-689A65DA: G***, kibuzzard-689A65DA, F.Cu at (126.4, 104.5)
- added kibuzzard-689A65F1: G***, kibuzzard-689A65F1, F.Cu at (135.3, 104.1)
- added kibuzzard-689A65FB: G***, kibuzzard-689A65FB, F.Cu at (136.0, 109.9)
- added kibuzzard-689A6605: G***, kibuzzard-689A6605, F.Cu at (129.3, 107.6)
- added kibuzzard-689A660E: G***, kibuzzard-689A660E, F.Cu at (128.3, 107.0)
- added kibuzzard-689A665F: G***, kibuzzard-689A665F, B.Cu at (136.8, 107.0)
- added kibuzzard-689A6665: G***, kibuzzard-689A6665, B.Cu at (133.9, 109.5)
- added kibuzzard-689A6668: G***, kibuzzard-689A6668, B.Cu at (132.5, 104.5)
- added kibuzzard-689A6672: G***, kibuzzard-689A6672, B.Cu at (128.3, 107.0)

Commit message: Update examples with latest parts
Parts:
- J1, J5: footprint SparkFun-Connector:1x01_1x1mm -> SparkFun-Connector:1x01_P2.0mm
- J2: footprint SparkFun-Connector:JST_SMD_1.0mm-4_Black -> SparkFun-Connector:JST_1x04_P1.0mm_Horizontal_SMD
- JP1: value ~ -> LED
- JP2: value ~ -> I2C
- JP3: value ~ -> ADR
Connections:
- U1 pad 2: (no net) -> NC2
- U1 pad 3: (no net) -> NC3
Changed lines of the file:
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@@
 	(net 16 "unconnected-(J2-NC-PadNC2)")
 	(net 17 "unconnected-(J2-NC-PadNC1)")
+	(net 18 "NC2")
+	(net 19 "NC3")
 	(footprint "kibuzzard-689A65FB"
 		(layer "F.Cu")
@@
 				(font
 					(size 0.001 0.001)
+					(thickness 0.15)
 				)
 			)
@@
 				(font
 					(size 0.001 0.001)
+					(thickness 0.15)
 				)
 			)
@@
 			)
 		)
-		(property "Datasheet" ""
+		(property "Datasheet" "~"
 			(at 0 0 0)
 			(unlocked yes)
@@
 			)
 		)
-		(property "PROD_ID" "RES-14241"
+		(property "PROD_ID" "RES-25567"
 			(at 0 0 0)
 			(unlocked yes)
@@
 		)
 	)
-	(footprint "SparkFun-Connector:1x01_1x1mm"
+	(footprint "SparkFun-Connector:1x01_P2.0mm"
 		(layer "F.Cu")
 		(at 128.346 104.456 180)
-		(descr "Plated Through Hole - No Silk Outline\n\nSpecifications:\n\n• Pin count:1\n• Pin pitch:0.1mm\n• Hole Size: .7mm\n• Annular Ring: 1.2mm\n\nMade for the small  https://www.sparkfun.com/products/18221  1mm Pitch Headers.")
 		(tags "SparkFun")
 		(property "Reference" "J5"
@@
 			)
 		)
-		(property "Datasheet" ""
+		(property "Datasheet" "~"
 			(at 0 0 180)
 			(layer "F.Fab")
@@
 				(font
 					(size 0.001 0.001)
+					(thickness 0.15)
 				)
 			)
@@
 				(font
 					(size 0.001 0.001)
+					(thickness 0.15)
 				)
 			)
@@
 				(font
 					(size 0.001 0.001)
+					(thickness 0.15)
 				)
 			)
@@
 				(font
 					(size 0.001 0.001)
+					(thickness 0.15)
 				)
 			)
@@
 		(embedded_fonts no)
 	)
-	(footprint "SparkFun-Connector:1x01_1x1mm"
+	(footprint "SparkFun-Connector:1x01_P2.0mm"
 		(layer "F.Cu")
 		(at 128.346 109.536 180)
-		(descr "Plated Through Hole - No Silk Outline\n\nSpecifications:\n\n• Pin count:1\n• Pin pitch:0.1mm\n• Hole Size: .7mm\n• Annular Ring: 1.2mm\n\nMade for the small  https://www.sparkfun.com/products/18221  1mm Pitch Headers.")
 		(tags "SparkFun")
 		(property "Reference" "J1"
@@
 			)
 		)
-		(property "Datasheet" ""
+		(property "Datasheet" "~"
 			(at 0 0 180)
 			(layer "F.Fab")
@@
 			)
 		)
-		(property "PROD_ID" "RES-14341"
+		(property "PROD_ID" "RES-25566"
 			(at 0 0 270)
 			(unlocked yes)
@@
 			)
 		)
-		(property "Datasheet" ""
+		(property "Datasheet" "~"
 			(at 0 0 0)
 			(unlocked yes)
@@
 			)
 		)
-		(property "PROD_ID" "CAP-15083"
+		(property "PROD_ID" "CAP-25565"
 			(at 0 0 180)
 			(unlocked yes)
@@
 			)
 		)
-		(property "Voltage" "10V"
+		(property "Voltage" "16V"
 			(at 0 0 180)
 			(unlocked yes)
@@
 				(font
 					(size 0.001 0.001)
+					(thickness 0.15)
 				)
 			)
@@
 				(font
 					(size 0.001 0.001)
+					(thickness 0.15)
 				)
 			)
@@
 			(size 0.7 0.28)
 			(layers "F.Cu" "F.Mask" "F.Paste")
+			(net 18 "NC2")
+			(pinfunction "NC2")
+			(pintype "power_in")
 			(solder_mask_margin 0.05)
 			(solder_paste_margin 0)
@@
 			(size 0.7 0.28)
 			(layers "F.Cu" "F.Mask" "F.Paste")
+			(net 19 "NC3")
+			(pinfunction "NC3")
+			(pintype "power_in")
 			(solder_mask_margin 0.05)
 			(solder_paste_margin 0)
@@
 		)
 	)
-	(footprint "SparkFun-Connector:JST_SMD_1.0mm-4_Black"
+	(footprint "SparkFun-Connector:JST_1x04_P1.0mm_Horizontal_SMD"
 		(layer "F.Cu")
 		(at 137.236 106.996 90)
@@
 		)
 		(property "Value" "Qwiic_RA"
-			(at 0 2.075 90)
+			(at 0 2.6 90)
 			(layer "F.Fab")
 			(effects
@@
 		)
 		(embedded_fonts no)
-		(model "${SPARKFUN_KICAD_LIBRARY}/Footprints/SparkFun-3D-models/Connector/Qwiic-Horizontal.STEP"
+		(model "${SPARKFUN_KICAD_LIBRARY}/3dmodels/Connector.3dshapes/Qwiic-Horizontal.step"
 			(offset
 				(xyz 0 -0.7 -0.3)
@@
 			)
 		)
-		(model "${SPARKFUN_KICAD_LIBRARY}/Footprints/SparkFun-3D-models/Connector/JST_SMD_1.0mm-4.STEP"
+		(model "${SPARKFUN_KICAD_LIBRARY}/3dmodels/Connector.3dshapes/JST_SMD_1.0mm-4.step"
 			(hide yes)
 			(offset
@@
 				(font
 					(size 0.001 0.001)
+					(thickness 0.15)
 				)
 			)
@@
 				(font
 					(size 0.001 0.001)
+					(thickness 0.15)
 				)
 			)
@@
 			)
 		)
-		(property "PROD_ID" "RES-14341"
+		(property "PROD_ID" "RES-25566"
 			(at 0 0 90)
 			(unlocked yes)
@@
 				(font
 					(size 0.001 0.001)
+					(thickness 0.15)
 				)
 			)
@@
 				(font
 					(size 0.001 0.001)
+					(thickness 0.15)
 				)
 			)
@@
 			)
 		)
-		(property "Datasheet" ""
+		(property "Datasheet" "~"
 			(at 0 0 0)
 			(unlocked yes)
@@
 			)
 		)
-		(property "Value" "~"
+		(property "Value" "ADR"
 			(at 0 -1.143 0)
 			(layer "B.Fab")
@@
 			)
 		)
-		(property "Datasheet" ""
+		(property "Datasheet" "~"
 			(at 0 0 0)
 			(unlocked yes)
@@
 			)
 		)
-		(property "Value" "~"
+		(property "Value" "I2C"
 			(at 0 -1.143 90)
 			(layer "B.Fab")
@@
 			)
 		)
-		(property "Datasheet" ""
+		(property "Datasheet" "~"
 			(at 0 0 90)
 			(unlocked yes)
@@
 			)
 		)
-		(property "Datasheet" ""
+		(property "Datasheet" "~"
 			(at 0 0 0)
 			(unlocked yes)
@@
 			)
 		)
-		(property "Datasheet" ""
+		(property "Datasheet" "~"
 			(at 0 0 0)
 			(unlocked yes)
@@
 			)
 		)
-		(property "Value" "~"
+		(property "Value" "LED"
 			(at 0 -1.143 0)
 			(layer "B.Fab")
@@
 			)
 		)
-		(property "Datasheet" ""
+		(property "Datasheet" "~"
 			(at 0 0 180)
 			(unlocked yes)
@@
 				(font
 					(size 0.001 0.001)
+					(thickness 0.15)
 				)
 				(justify mirror)
@@
 				(font
 					(size 0.001 0.001)
+					(thickness 0.15)
 				)
 				(justify mirror)
@@
 			)
 		)
-		(property "Datasheet" ""
+		(property "Datasheet" "~"
 			(at 0 0 0)
 			(unlocked yes)
@@
 				(font
 					(size 0.001 0.001)
+					(thickness 0.15)
 				)
 				(justify mirror)
@@
 				(font
 					(size 0.001 0.001)
+					(thickness 0.15)
 				)
 				(justify mirror)
@@
 				(font
 					(size 0.001 0.001)
+					(thickness 0.15)
 				)
 				(justify mirror)
@@
 				(font
 					(size 0.001 0.001)
+					(thickness 0.15)
 				)
 				(justify mirror)
@@
 			)
 		)
-		(property "Datasheet" ""
+		(property "Datasheet" "~"
 			(at 0 0 0)
 			(unlocked yes)
@@
 				(font
 					(size 0.001 0.001)
+					(thickness 0.15)
 				)
 				(justify mirror)
@@
 				(font
 					(size 0.001 0.001)
+					(thickness 0.15)
 				)
 				(justify mirror)
@@
 			(keep_text_aligned yes)
 		)
-		(gr_text "750 mils"
+		(gr_text "19.05 mm"
 			(at 132.791 98.1585 0)
 			(layer "Dwgs.User")
@@
 			(keep_text_aligned yes)
 		)
-		(gr_text "200 mils"
+		(gr_text "5.08 mm"
 			(at 125.806 101.3335 0)
 			(layer "Dwgs.User")
@@
 			(keep_text_aligned yes)
 		)
-		(gr_text "300 mils"
+		(gr_text "7.62 mm"
 			(at 143.956 106.996 90)
 			(layer "Dwgs.User")
@@
 			(keep_text_aligned yes)
 		)
-		(gr_text "50 mils"
+		(gr_text "1.27 mm"
 			(at 119.202 103.948 90)
 			(layer "Dwgs.User")
@@
 			(keep_text_aligned yes)
 		)
-		(gr_text "100 mils"
+		(gr_text "2.54 mm"
 			(at 124.536 113.346 0)
 			(layer "Dwgs.User")
