File: Example-Qwiic Micro Breakout/SparkFun_Example_Micro.kicad_sch (KiCad schematic)
At the start: 23 parts, among them J1 PTH_1x1mm, J2 Qwiic_RA, J5 PTH_1x1mm

Commit message: Remove duplicate files
Parts:
- added C4: 10uF, SparkFun-Capacitor:C_0402_1005Metric, symbol SparkFun-Capacitor:10uF_0402_6.3V_20%
- added JP3: ADDR, SparkFun-Jumper:Jumper_2_NO, symbol SparkFun-Jumper:SolderJumper_2_Open
- added R2: 10k, SparkFun-Resistor:R_0402_1005Metric, symbol SparkFun-Resistor:10k_0402
- added U1: LIS3DH, SparkFun-Sensor:ST_LGA-16_3x3mm_P0.5mm_5x3, symbol SparkFun-Sensor:LIS3DH
- D1: footprint SparkFun-LED:LED_0402_1005Metric -> SparkFun-LED:LED_0402_1005Metric_Red; PROD_ID DIO-25000 -> DIO-16757
- J1, J5: footprint SparkFun-Connector:1x01_PTH_1x1mm -> SparkFun-Connector:1x01_1x1mm
Connections:
- net 3.3V: now also C4.1, R2.2, U1.1 (VDDIO), U1.14 (VDD)
- net GND: now also C4.2, JP3.1 (A), U1.10 (RES), U1.12 (GND), U1.5 (GND)
- net SCL: now also U1.4 (SCL/SPC)
- net SDA: now also U1.6 (SDA/SDI)
- net INT renamed INT1
- net INT1: now also U1.11 (INT1)
- new net ADDR/SDO: JP3.2 (B), R2.1, U1.7 (SA0/SDO)
- no-connect marks 0 -> 5
Other:
- note added: "Close "ADDR" Jumper to Change Address to 0x18"
- note added: "Plated through holes can fit 22AWG wire or smaller."
- title: SparkFun  Sensor -  -> SparkFun Triple Axis Accelerometer - LIS3DH
- moved on the sheet: C3

Commit message: Add axis labels
Parts:
- removed FID1, FID2: Fiducial_0.5mm, SparkFun-Aesthetic:Fiducial_0.5mm_Mask1mm, symbol SparkFun-Aesthetic:Fiducial_0.5mm
- J1, J5: footprint SparkFun-Connector:1x01_1x1mm -> SparkFun-Connector:1x01_PTH_1x1mm
- JP1: value LED -> ~
- JP2: value I2C -> ~
- JP3: value ADDR -> ~
Connections:
- net ADDR/SDO renamed ADR/SDO
Other:
- note added: "Close "ADR" jumper to change address to 0x18"
- note added: "Cut jumper to remove pull-up resistors"
- note added: "Default 7-bit unshifted I²C address: 0x19"
- note removed: "Close "ADDR" Jumper to Change Address to 0x18"
- note removed: "Cut jumper to remove pull-up resistors."
- note removed: "Default 7-bit Unshifted Address: 0x19"

Commit message: Make labels and text follow standard
Parts:
- JP1: value ~ -> LED
- JP2: value ~ -> I2C
- JP3: value ~ -> ADR
Changed lines of the file:
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@@
 				)
 				(justify right)
-			)
-		)
-		(property "Value" "~"
-			(at 137.16 71.12 90)
+				(hide yes)
+			)
+		)
+		(property "Value" "ADR"
+			(at 137.16 69.8499 90)
 			(effects
 				(font
@@
 			)
 		)
-		(property "Value" "~"
+		(property "Value" "I2C"
 			(at 210.82 127 0)
 			(effects
@@
 			)
 		)
-		(property "Value" "~"
+		(property "Value" "LED"
 			(at 212.598 58.674 90)
 			(effects

Commit message: Update examples with latest parts
Parts:
- C3: symbol SparkFun-Capacitor:0.1uF_0402_10V_10% -> SparkFun-Capacitor:0.1uF_0402_16V_10%; PROD_ID CAP-15083 -> CAP-25565; Voltage 10V -> 16V
- J1, J5: footprint SparkFun-Connector:1x01_PTH_1x1mm -> SparkFun-Connector:1x01_P2.0mm; symbol SparkFun-Connector:Conn_01x01_PTH_1x1mm -> SparkFun-Connector:Conn_01x01_P2.0mm
- J2: footprint SparkFun-Connector:JST_SMD_1.0mm-4_Black -> SparkFun-Connector:JST_1x04_P1.0mm_Horizontal_SMD; symbol SparkFun-Connector:Qwiic_Right_Angle -> SparkFun-Connector:Qwiic_Horizontal
- R1, R6: PROD_ID RES-14341 -> RES-25566
- R2: PROD_ID RES-14241 -> RES-25567
Connections:
- new net NC2: U1.2 (NC2)
- new net NC3: U1.3 (NC3)
Changed lines of the file:
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@@
 		(effects
 			(font
-				(size 2.54 2.54)
+				(size 3 3)
 			)
 		)
@@
 	)
 	(global_label "INT1"
-		(shape input)
+		(shape output)
 		(at 100.33 137.16 180)
 		(fields_autoplaced yes)
@@
 	)
 	(global_label "INT1"
-		(shape input)
+		(shape output)
 		(at 96.52 71.12 0)
 		(fields_autoplaced yes)
@@
 			)
 		)
-		(property "PROD_ID" "RES-14241"
+		(property "PROD_ID" "RES-25567"
 			(at 140.97 62.23 0)
 			(effects
@@
 	)
 	(symbol
-		(lib_id "SparkFun-Connector:Qwiic_Right_Angle")
+		(lib_id "SparkFun-Connector:Qwiic_Horizontal")
 		(at 72.39 137.16 0)
 		(unit 1)
@@
 			)
 		)
-		(property "Footprint" "SparkFun-Connector:JST_SMD_1.0mm-4_Black"
+		(property "Footprint" "SparkFun-Connector:JST_1x04_P1.0mm_Horizontal_SMD"
 			(at 72.39 149.86 0)
 			(effects
@@
 	)
 	(symbol
-		(lib_id "SparkFun-Connector:Conn_01x01_PTH_1x1mm")
+		(lib_id "SparkFun-Connector:Conn_01x01_P2.0mm")
 		(at 106.68 139.7 0)
 		(unit 1)
@@
 			)
 		)
-		(property "Footprint" "SparkFun-Connector:1x01_PTH_1x1mm"
+		(property "Footprint" "SparkFun-Connector:1x01_P2.0mm"
 			(at 106.68 147.32 0)
 			(effects
@@
 	)
 	(symbol
-		(lib_id "SparkFun-Capacitor:0.1uF_0402_10V_10%")
+		(lib_id "SparkFun-Capacitor:0.1uF_0402_16V_10%")
 		(at 55.88 64.77 0)
 		(unit 1)
@@
 			)
 		)
-		(property "PROD_ID" "CAP-15083"
+		(property "PROD_ID" "CAP-25565"
 			(at 55.88 81.28 0)
 			(effects
@@
 			)
 		)
-		(property "Voltage" "10V"
+		(property "Voltage" "16V"
 			(at 58.42 66.0462 0)
 			(effects
@@
 			)
 		)
-		(property "PROD_ID" "RES-14341"
+		(property "PROD_ID" "RES-25566"
 			(at 221.488 128.27 0)
 			(effects
@@
 	)
 	(symbol
-		(lib_id "SparkFun-Connector:Conn_01x01_PTH_1x1mm")
+		(lib_id "SparkFun-Connector:Conn_01x01_P2.0mm")
 		(at 106.68 137.16 0)
 		(unit 1)
@@
 			)
 		)
-		(property "Footprint" "SparkFun-Connector:1x01_PTH_1x1mm"
+		(property "Footprint" "SparkFun-Connector:1x01_P2.0mm"
 			(at 106.68 144.78 0)
 			(effects
@@
 		(pin "8"
 		)
+		(pin "2"
+		)
+		(pin "3"
+		)
 		(instances
 			(project ""
@@
 		(dnp no)
 		(property "Reference" "R1"
-			(at 201.422 127 90)
+			(at 201.93 127 90)
 			(effects
 				(font
@@
 		)
 		(property "Value" "2.2k"
-			(at 201.422 129.54 90)
+			(at 200.66 129.54 90)
 			(effects
 				(font
@@
 			)
 		)
-		(property "PROD_ID" "RES-14341"
+		(property "PROD_ID" "RES-25566"
 			(at 213.868 128.27 0)
 			(effects
